File: MicroFLiC_junction_shield_1_0.sch (KiCad schematic (older format))
At the start: 46 parts, among them P1 14-way Micro-MaTch, P2 8-way Micro-MaTch, P3 6-way Micro-MaTch, P4 12-way Micro-MaTch, P5 1x4 Socket Strip R/A, SW1 Tactile Switch R/A, U1 23LCV1024

Commit message: Last commit in v1.0
Parts:
- R3, R4, R5: Order COde 2447551 -> (none); Order Code (none) -> 2447551
Changed lines of the file:
@@
 F 4 "MCWR08X1003FTL" V 10400 1400 60  0001 C CNN "Part Number"
 F 5 "Multicomp" V 10400 1400 60  0001 C CNN "Manufacturer"
-F 6 "2447551" V 10400 1400 60  0001 C CNN "Order COde"
+F 6 "2447551" V 10400 1400 60  0001 C CNN "Order Code"
 	1    10400 1400
 	0    1    1    0
@@
 F 4 "MCWR08X1003FTL" V 10400 1600 60  0001 C CNN "Part Number"
 F 5 "Multicomp" V 10400 1600 60  0001 C CNN "Manufacturer"
-F 6 "2447551" V 10400 1600 60  0001 C CNN "Order COde"
+F 6 "2447551" V 10400 1600 60  0001 C CNN "Order Code"
 	1    10400 1600
 	0    1    1    0
@@
 F 4 "MCWR08X1003FTL" V 10400 1800 60  0001 C CNN "Part Number"
 F 5 "Multicomp" V 10400 1800 60  0001 C CNN "Manufacturer"
-F 6 "2447551" V 10400 1800 60  0001 C CNN "Order COde"
+F 6 "2447551" V 10400 1800 60  0001 C CNN "Order Code"
 	1    10400 1800
 	0    1    1    0
