File: LCDandRTC.sch (KiCad schematic (older format))
At the start: 13 parts, among them P6 2x8 socket strip, Q3 TSM2314, U2 PCA9306DP, U3 DS1338, X1 32.768kHz

Commit message: Last commit in v1.0
Parts:
- R10: Order COde 2447551 -> (none); Order Code (none) -> 2447551
Other:
- note removed: "TTL buffers for 3.3V to 5V level shifting"
Changed lines of the file:
@@
 P 4200 5650
 F 0 "P6" H 4200 6100 50  0000 C CNN
-F 1 "2x8 socket strip" V 4200 5650 50  0000 C CNN
+F 1 "2x8 socket strip" H 4200 5200 50  0000 C CNN
 F 2 "Socket_Strips:Socket_Strip_Straight_2x08" H 4200 4450 50  0001 C CNN
 F 3 "" H 4200 4450 50  0000 C CNN
@@
 L GND #PWR034
 U 1 1 566AD7CE
-P 3850 6100
-F 0 "#PWR034" H 3850 5850 50  0001 C CNN
-F 1 "GND" H 3850 5950 50  0000 C CNN
-F 2 "" H 3850 6100 50  0000 C CNN
-F 3 "" H 3850 6100 50  0000 C CNN
-	1    3850 6100
+P 3750 6100
+F 0 "#PWR034" H 3750 5850 50  0001 C CNN
+F 1 "GND" H 3750 5950 50  0000 C CNN
+F 2 "" H 3750 6100 50  0000 C CNN
+F 3 "" H 3750 6100 50  0000 C CNN
+	1    3750 6100
 	1    0    0    -1
 $EndComp
@@
 F 4 "MCWR08X1003FTL" V 5200 3250 60  0001 C CNN "Part Number"
 F 5 "Multicomp" V 5200 3250 60  0001 C CNN "Manufacturer"
-F 6 "2447551" V 5200 3250 60  0001 C CNN "Order COde"
+F 6 "2447551" V 5200 3250 60  0001 C CNN "Order Code"
 	1    5200 3250
 	-1   0    0    1
@@
 	4450 5700 5050 5700
 Wire Wire Line
-	3950 6000 3850 6000
-Wire Wire Line
-	3850 6000 3850 6100
+	3950 6000 3750 6000
+Wire Wire Line
+	3750 6000 3750 6100
 Wire Wire Line
 	4450 5500 5050 5500
@@
 Wire Wire Line
 	5200 3100 5200 3000
-Text Notes 4050 4100 0    60   ~ 0
-TTL buffers for 3.3V to 5V level shifting
 Text HLabel 3350 5300 0    60   Input ~ 0
 LCD_A0

Commit message: Finished adding full part descriptions
Parts:
- C5, C6, C7: Alt. Order Code (none) -> 710-885012207098; Alt. Supplier (none) -> Mouser; Note (none) -> 100nF/50V X7R 0805 ceramic capacitor; Package (none) -> 0805; Supplier (none) -> Farnell
- P6: Alt. Order Code (none) -> ESQ-108-33-G-D; Alt. Supplier (none) -> Samtec; Note (none) -> 2x8 ESQ series elevated socket strip; Package (none) -> DIL-16; Supplier (none) -> Farnell
- Q3: Alt. Order Code (none) -> 781-SI2314EDS-E3; Alt. Supplier (none) -> Mouser; Note (none) -> N-channel SOT-23 MOSFET; Package (none) -> SOT-23; Supplier (none) -> Farnell
- R10, R11: Alt. Order Code (none) -> 71-CRCW0805-100K-E3; Alt. Supplier (none) -> Mouser; Note (none) -> 100kΩ/1% 0805 resistor; Package (none) -> 0805; Supplier (none) -> Farnell
- R12, R8, R9: Alt. Order Code (none) -> 71-CRCW0805-1.5K-E3; Alt. Supplier (none) -> Mouser; Note (none) -> 1.5kΩ/1% 0805 resistor; Package (none) -> 0805; Supplier (none) -> Farnell
- U2: Alt. Order Code (none) -> 771-PCA9306DP-T; Alt. Supplier (none) -> Mouser; Note (none) -> Dual I²C-bus voltage translator; Package (none) -> TSSOP-8; Supplier (none) -> Farnell
- U3: Alt. Order Code (none) -> 700-DS1338Z-33; Alt. Supplier (none) -> Mouser; Note (none) -> I²C real time clock with NVRAM; Package (none) -> SOIC-8; Supplier (none) -> Farnell
- X1: Alt. Order Code (none) -> 559-FSRLF327; Alt. Supplier (none) -> Mouser; Note (none) -> 32.768kHz 12.5pF crystal; Package (none) -> 8.7mm×3.7mm; Supplier (none) -> Farnell
Changed lines of the file:
@@
 F 4 "PCA9306DP" H 4250 2200 60  0001 C CNN "Part Number"
 F 5 "NXP" H 4250 2200 60  0001 C CNN "Manufacturer"
-F 6 "2212072" H 4250 2200 60  0001 C CNN "Order Code"
+F 6 "TSSOP-8" H 4250 2200 60  0001 C CNN "Package"
+F 7 "Farnell" H 4250 2200 60  0001 C CNN "Supplier"
+F 8 "2212072" H 4250 2200 60  0001 C CNN "Order Code"
+F 9 "Mouser" H 4250 2200 60  0001 C CNN "Alt. Supplier"
+F 10 "771-PCA9306DP-T" H 4250 2200 60  0001 C CNN "Alt. Order Code"
+F 11 "Dual I²C-bus voltage translator" H 4250 2200 60  0001 C CNN "Note"
 	1    4250 2200
 	1    0    0    -1
@@
 F 4 "MCWR08X1003FTL" V 6550 2000 60  0001 C CNN "Part Number"
 F 5 "Multicomp" V 6550 2000 60  0001 C CNN "Manufacturer"
-F 6 "2447551" V 6550 2000 60  0001 C CNN "Order Code"
+F 6 "0805" H 6550 2000 60  0001 C CNN "Package"
+F 7 "Farnell" H 6550 2000 60  0001 C CNN "Supplier"
+F 8 "2447551" V 6550 2000 60  0001 C CNN "Order Code"
+F 9 "Mouser" H 6550 2000 60  0001 C CNN "Alt. Supplier"
+F 10 "71-CRCW0805-100K-E3" H 6550 2000 60  0001 C CNN "Alt. Order Code"
+F 11 "100kΩ/1% 0805 resistor" H 6550 2000 60  0001 C CNN "Note"
 	1    6550 2000
 	0    1    1    0
@@
 F 4 "TSM2314CX" H 6200 3500 60  0001 C CNN "Part Number"
 F 5 "Taiwan Semiconductor" H 6200 3500 60  0001 C CNN "Manufacturer"
-F 6 "1864589" H 6200 3500 60  0001 C CNN "Order Code"
+F 6 "SOT-23" H 6200 3500 60  0001 C CNN "Package"
+F 7 "Farnell" H 6200 3500 60  0001 C CNN "Supplier"
+F 8 "1864589" H 6200 3500 60  0001 C CNN "Order Code"
+F 9 "Mouser" H 6200 3500 60  0001 C CNN "Alt. Supplier"
+F 10 "781-SI2314EDS-E3" H 6200 3500 60  0001 C CNN "Alt. Order Code"
+F 11 "N-channel SOT-23 MOSFET" H 6200 3500 60  0001 C CNN "Note"
 	1    6200 3500
 	1    0    0    -1
@@
 F 4 "MCWR08X1501FTL" V 5000 1350 60  0001 C CNN "Part Number"
 F 5 "Multicomp" V 5000 1350 60  0001 C CNN "Manufacturer"
-F 6 "2447592" V 5000 1350 60  0001 C CNN "Order Code"
+F 6 "0805" H 5000 1350 60  0001 C CNN "Package"
+F 7 "Farnell" H 5000 1350 60  0001 C CNN "Supplier"
+F 8 "2447592" V 5000 1350 60  0001 C CNN "Order Code"
+F 9 "Mouser" H 5000 1350 60  0001 C CNN "Alt. Supplier"
+F 10 "71-CRCW0805-1.5K-E3" H 5000 1350 60  0001 C CNN "Alt. Order Code"
+F 11 "1.5kΩ/1% 0805 resistor" H 5000 1350 60  0001 C CNN "Note"
 	1    5000 1350
 	-1   0    0    1
@@
 F 4 "ESQ-108-33-G-D" H 4200 5650 60  0001 C CNN "Part Number"
 F 5 "Samtec" H 4200 5650 60  0001 C CNN "Manufacturer"
-F 6 "1930550" H 4200 5650 60  0001 C CNN "Order Code"
+F 6 "DIL-16" H 4200 5650 60  0001 C CNN "Package"
+F 7 "Farnell" H 4200 5650 60  0001 C CNN "Supplier"
+F 8 "1930550" H 4200 5650 60  0001 C CNN "Order Code"
+F 9 "Samtec" H 4200 5650 60  0001 C CNN "Alt. Supplier"
+F 10 "ESQ-108-33-G-D" H 4200 5650 60  0001 C CNN "Alt. Order Code"
+F 11 "2x8 ESQ series elevated socket strip" H 4200 5650 60  0001 C CNN "Note"
 	1    4200 5650
 	1    0    0    -1
@@
 F 4 "DS1338Z-33" H 9100 2300 60  0001 C CNN "Part Number"
 F 5 "Maxim Integrated" H 9100 2300 60  0001 C CNN "Manufacturer"
-F 6 "1379714" H 9100 2300 60  0001 C CNN "Order Code"
+F 6 "SOIC-8" H 9100 2300 60  0001 C CNN "Package"
+F 7 "Farnell" H 9100 2300 60  0001 C CNN "Supplier"
+F 8 "1379714" H 9100 2300 60  0001 C CNN "Order Code"
+F 9 "Mouser" H 9100 2300 60  0001 C CNN "Alt. Supplier"
+F 10 "700-DS1338Z-33" H 9100 2300 60  0001 C CNN "Alt. Order Code"
+F 11 "I²C real time clock with NVRAM" H 9100 2300 60  0001 C CNN "Note"
 	1    9100 2300
 	1    0    0    -1
@@
 F 4 "FSRLF327" H 8050 2450 60  0001 C CNN "Part Number"
 F 5 "Fox Electronics" H 8050 2450 60  0001 C CNN "Manufacturer"
-F 6 "2064035" H 8050 2450 60  0001 C CNN "Order Code"
+F 6 "8.7mm×3.7mm" H 8050 2450 60  0001 C CNN "Package"
+F 7 "Farnell" H 8050 2450 60  0001 C CNN "Supplier"
+F 8 "2064035" H 8050 2450 60  0001 C CNN "Order Code"
+F 9 "Mouser" H 8050 2450 60  0001 C CNN "Alt. Supplier"
+F 10 "559-FSRLF327" H 8050 2450 60  0001 C CNN "Alt. Order Code"
+F 11 "32.768kHz 12.5pF crystal" H 8050 2450 60  0001 C CNN "Note"
 	1    8050 2450
 	1    0    0    -1
@@
 F 4 "MCWR08X1003FTL" V 5200 3250 60  0001 C CNN "Part Number"
 F 5 "Multicomp" V 5200 3250 60  0001 C CNN "Manufacturer"
-F 6 "2447551" V 5200 3250 60  0001 C CNN "Order Code"
+F 6 "0805" H 5200 3250 60  0001 C CNN "Package"
+F 7 "Farnell" H 5200 3250 60  0001 C CNN "Supplier"
+F 8 "2447551" V 5200 3250 60  0001 C CNN "Order Code"
+F 9 "Mouser" H 5200 3250 60  0001 C CNN "Alt. Supplier"
+F 10 "71-CRCW0805-100K-E3" H 5200 3250 60  0001 C CNN "Alt. Order Code"
+F 11 "100kΩ/1% 0805 resistor" H 5200 3250 60  0001 C CNN "Note"
 	1    5200 3250
 	-1   0    0    1
@@
 F 4 "MC0805B104K250CT" H 5400 1350 60  0001 C CNN "Part Number"
 F 5 "Multicomp" H 5400 1350 60  0001 C CNN "Manufacturer"
-F 6 "1759166" H 5400 1350 60  0001 C CNN "Order Code"
+F 6 "0805" H 5400 1350 60  0001 C CNN "Package"
+F 7 "Farnell" H 5400 1350 60  0001 C CNN "Supplier"
+F 8 "1759166" H 5400 1350 60  0001 C CNN "Order Code"
+F 9 "Mouser" H 5400 1350 60  0001 C CNN "Alt. Supplier"
+F 10 "710-885012207098" H 5400 1350 60  0001 C CNN "Alt. Order Code"
+F 11 "100nF/50V X7R 0805 ceramic capacitor" H 5400 1350 60  0001 C CNN "Note"
 	1    5400 1350
 	1    0    0    -1
@@
 F 4 "MC0805B104K250CT" H 10600 1750 60  0001 C CNN "Part Number"
 F 5 "Multicomp" H 10600 1750 60  0001 C CNN "Manufacturer"
-F 6 "1759166" H 10600 1750 60  0001 C CNN "Order Code"
+F 6 "0805" H 10600 1750 60  0001 C CNN "Package"
+F 7 "Farnell" H 10600 1750 60  0001 C CNN "Supplier"
+F 8 "1759166" H 10600 1750 60  0001 C CNN "Order Code"
+F 9 "Mouser" H 10600 1750 60  0001 C CNN "Alt. Supplier"
+F 10 "710-885012207098" H 10600 1750 60  0001 C CNN "Alt. Order Code"
+F 11 "100nF/50V X7R 0805 ceramic capacitor" H 10600 1750 60  0001 C CNN "Note"
 	1    10600 1750
 	1    0    0    -1
@@
 F 4 "MC0805B104K250CT" H 6800 2400 60  0001 C CNN "Part Number"
 F 5 "Multicomp" H 6800 2400 60  0001 C CNN "Manufacturer"
-F 6 "1759166" H 6800 2400 60  0001 C CNN "Order Code"
+F 6 "0805" H 6800 2400 60  0001 C CNN "Package"
+F 7 "Farnell" H 6800 2400 60  0001 C CNN "Supplier"
+F 8 "1759166" H 6800 2400 60  0001 C CNN "Order Code"
+F 9 "Mouser" H 6800 2400 60  0001 C CNN "Alt. Supplier"
+F 10 "710-885012207098" H 6800 2400 60  0001 C CNN "Alt. Order Code"
+F 11 "100nF/50V X7R 0805 ceramic capacitor" H 6800 2400 60  0001 C CNN "Note"
 	1    6800 2400
 	1    0    0    -1
@@
 F 4 "MCWR08X1501FTL" V 5200 1350 60  0001 C CNN "Part Number"
 F 5 "Multicomp" V 5200 1350 60  0001 C CNN "Manufacturer"
-F 6 "2447592" V 5200 1350 60  0001 C CNN "Order Code"
+F 6 "0805" H 5200 1350 60  0001 C CNN "Package"
+F 7 "Farnell" H 5200 1350 60  0001 C CNN "Supplier"
+F 8 "2447592" V 5200 1350 60  0001 C CNN "Order Code"
+F 9 "Mouser" H 5200 1350 60  0001 C CNN "Alt. Supplier"
+F 10 "71-CRCW0805-1.5K-E3" H 5200 1350 60  0001 C CNN "Alt. Order Code"
+F 11 "1.5kΩ/1% 0805 resistor" H 5200 1350 60  0001 C CNN "Note"
 	1    5200 1350
 	-1   0    0    1
@@
 F 4 "MCWR08X1501FTL" V 6800 1750 60  0001 C CNN "Part Number"
 F 5 "Multicomp" V 6800 1750 60  0001 C CNN "Manufacturer"
-F 6 "2447592" V 6800 1750 60  0001 C CNN "Order Code"
+F 6 "0805" H 6800 1750 60  0001 C CNN "Package"
+F 7 "Farnell" H 6800 1750 60  0001 C CNN "Supplier"
+F 8 "2447592" V 6800 1750 60  0001 C CNN "Order Code"
+F 9 "Mouser" H 6800 1750 60  0001 C CNN "Alt. Supplier"
+F 10 "71-CRCW0805-1.5K-E3" H 6800 1750 60  0001 C CNN "Alt. Order Code"
+F 11 "1.5kΩ/1% 0805 resistor" H 6800 1750 60  0001 C CNN "Note"
 	1    6800 1750
 	-1   0    0    1

Commit message: Incorporated un-pulled changes
Parts:
- U2: value PCA9306DP -> PCA9306; Manufacturer NXP -> NXP Semiconductors
Changed lines of the file:
@@
 P 4250 2200
 F 0 "U2" H 4250 2700 60  0000 C CNN
-F 1 "PCA9306DP" H 4250 2600 60  0000 C CNN
+F 1 "PCA9306" H 4250 2600 60  0000 C CNN
 F 2 "Housings_SSOP:MSOP-8_3x3mm_Pitch0.65mm" H 4250 2200 60  0001 C CNN
 F 3 "" H 4250 2200 60  0000 C CNN
 F 4 "PCA9306DP" H 4250 2200 60  0001 C CNN "Part Number"
-F 5 "NXP" H 4250 2200 60  0001 C CNN "Manufacturer"
+F 5 "NXP Semiconductors" H 4250 2200 60  0001 C CNN "Manufacturer"
 F 6 "TSSOP-8" H 4250 2200 60  0001 C CNN "Package"
 F 7 "Farnell" H 4250 2200 60  0001 C CNN "Supplier"
