File: LCDandRTC.sch (KiCad schematic (older format))
At the start: 13 parts, among them P6 2x8 socket strip, Q3 TSM2314, U2 PCA9306, U3 DS1338, X1 32.768kHz

Commit message: Changed LCD shield from Wire to Wire1
Connections:
- net labels added: I2C_EN, SCL1, SDA1
- net labels removed: SCL, SDA
Changed lines of the file:
@@
 EESchema Schematic File Version 2
-LIBS:MicroFLiC_junction_shield-rescue
 LIBS:power
 LIBS:device
@@
 $EndComp
 Text Label 3200 2450 0    60   ~ 0
-SDA
+SDA1
 Text Label 3200 2300 0    60   ~ 0
-SCL
-$Comp
-L +3V3 #PWR27
+SCL1
+$Comp
+L +3V3 #PWR031
 U 1 1 566ACC96
 P 3500 1900
-F 0 "#PWR27" H 3500 1750 50  0001 C CNN
+F 0 "#PWR031" H 3500 1750 50  0001 C CNN
 F 1 "+3V3" H 3500 2040 50  0000 C CNN
 F 2 "" H 3500 1900 50  0000 C CNN
@@
 $EndComp
 $Comp
-L +5V #PWR35
+L +5V #PWR032
 U 1 1 566ACCAB
 P 6800 1500
-F 0 "#PWR35" H 6800 1350 50  0001 C CNN
+F 0 "#PWR032" H 6800 1350 50  0001 C CNN
 F 1 "+5V" H 6800 1640 50  0000 C CNN
 F 2 "" H 6800 1500 50  0000 C CNN
@@
 $EndComp
 $Comp
-L GND #PWR34
+L GND #PWR033
 U 1 1 566ACCC2
 P 6250 2700
-F 0 "#PWR34" H 6250 2450 50  0001 C CNN
+F 0 "#PWR033" H 6250 2450 50  0001 C CNN
 F 1 "GND" H 6250 2550 50  0000 C CNN
 F 2 "" H 6250 2700 50  0000 C CNN
@@
 $EndComp
 $Comp
-L GND #PWR29
+L GND #PWR034
 U 1 1 566ACCCF
 P 4250 3100
-F 0 "#PWR29" H 4250 2850 50  0001 C CNN
+F 0 "#PWR034" H 4250 2850 50  0001 C CNN
 F 1 "GND" H 4250 2950 50  0000 C CNN
 F 2 "" H 4250 3100 50  0000 C CNN
@@
 $EndComp
 $Comp
-L GND #PWR36
+L GND #PWR035
 U 1 1 566ACCD5
 P 6800 3800
-F 0 "#PWR36" H 6800 3550 50  0001 C CNN
+F 0 "#PWR035" H 6800 3550 50  0001 C CNN
 F 1 "GND" H 6800 3650 50  0000 C CNN
 F 2 "" H 6800 3800 50  0000 C CNN
@@
 $EndComp
 $Comp
-L +5V #PWR31
+L +5V #PWR036
 U 1 1 566ACCFE
 P 5200 1000
-F 0 "#PWR31" H 5200 850 50  0001 C CNN
+F 0 "#PWR036" H 5200 850 50  0001 C CNN
 F 1 "+5V" H 5200 1140 50  0000 C CNN
 F 2 "" H 5200 1000 50  0000 C CNN
@@
 $EndComp
 $Comp
-L GND #PWR33
+L GND #PWR037
 U 1 1 566ACD0E
 P 5400 1600
-F 0 "#PWR33" H 5400 1350 50  0001 C CNN
+F 0 "#PWR037" H 5400 1350 50  0001 C CNN
 F 1 "GND" H 5400 1450 50  0000 C CNN
 F 2 "" H 5400 1600 50  0000 C CNN
@@
 $EndComp
 Text HLabel 3100 2450 0    60   BiDi ~ 0
-SDA
+SDA1
 Text HLabel 3100 2300 0    60   BiDi ~ 0
-SCL
+SCL1
 Text HLabel 3100 3500 0    60   Input ~ 0
 ~I2C_EN
@@
 LCD_D5
 $Comp
-L GND #PWR28
+L GND #PWR038
 U 1 1 566AD7CE
 P 3750 6100
-F 0 "#PWR28" H 3750 5850 50  0001 C CNN
+F 0 "#PWR038" H 3750 5850 50  0001 C CNN
 F 1 "GND" H 3750 5950 50  0000 C CNN
 F 2 "" H 3750 6100 50  0000 C CNN
@@
 $EndComp
 $Comp
-L +BATT #PWR39
+L +BATT #PWR039
 U 1 1 566ADC91
 P 10100 2450
-F 0 "#PWR39" H 10100 2300 50  0001 C CNN
+F 0 "#PWR039" H 10100 2300 50  0001 C CNN
 F 1 "+BATT" V 10100 2590 50  0000 L CNN
 F 2 "" H 10100 2450 50  0000 C CNN
@@
 $EndComp
 $Comp
-L +3V3 #PWR32
+L +3V3 #PWR040
 U 1 1 566B2C19
 P 5200 3000
-F 0 "#PWR32" H 5200 2850 50  0001 C CNN
+F 0 "#PWR040" H 5200 2850 50  0001 C CNN
 F 1 "+3V3" H 5200 3140 50  0000 C CNN
 F 2 "" H 5200 3000 50  0000 C CNN
@@
 NoConn ~ 9900 2150
 $Comp
-L +12V #PWR30
+L +12V #PWR041
 U 1 1 566AAE29
 P 4650 5200
-F 0 "#PWR30" H 4650 5050 50  0001 C CNN
+F 0 "#PWR041" H 4650 5050 50  0001 C CNN
 F 1 "+12V" H 4650 5340 50  0000 C CNN
 F 2 "" H 4650 5200 50  0000 C CNN
@@
 	9100 1550 9100 1300
 $Comp
-L +5V #PWR37
+L +5V #PWR042
 U 1 1 56700AB7
 P 9100 1300
-F 0 "#PWR37" H 9100 1150 50  0001 C CNN
+F 0 "#PWR042" H 9100 1150 50  0001 C CNN
 F 1 "+5V" H 9100 1440 50  0000 C CNN
 F 2 "" H 9100 1300 50  0000 C CNN
@@
 $EndComp
 $Comp
-L GND #PWR38
+L GND #PWR043
 U 1 1 56700B0D
 P 9100 3300
-F 0 "#PWR38" H 9100 3050 50  0001 C CNN
+F 0 "#PWR043" H 9100 3050 50  0001 C CNN
 F 1 "GND" H 9100 3150 50  0000 C CNN
 F 2 "" H 9100 3300 50  0000 C CNN
@@
 	-1   0    0    1
 $EndComp
+Text Label 5300 2000 0    60   ~ 0
+I2C_EN
 $EndSCHEMATC
