File: MicroFLiC_junction_shield.sch (KiCad schematic (older format))
At the start: 46 parts, among them P1 14-way Micro-MaTch, P2 8-way Micro-MaTch, P3 6-way Micro-MaTch, P4 12-way Micro-MaTch, P5 1x4 Socket Strip R/A, SW1 Tactile Switch R/A, U1 23LCV1024

Commit message: Started fully describing components
Parts:
- C1, C2, C3: Alt. Order Code (none) -> 710-885012207098; Alt. Supplier (none) -> Mouser; Note (none) -> 100nF/50V X7R 0805 ceramic capacitor; Package (none) -> 0805; Supplier (none) -> Farnell
- P1: Alt. Order Code (none) -> 571-8-188275-4; Alt. Supplier (none) -> Mouser; Note (none) -> 14-way SMD Micro-MaTch connector; Order Code (none) -> 3784769; Package (none) -> Micro-MaTch SMD; Part Number 3784769 -> 8-188275-4; Supplier (none) -> Farnell
- P2: Alt. Order Code (none) -> 571-7-188275-8; Alt. Supplier (none) -> Mouser; Note (none) -> 8-way SMD Micro-MaTch connector; Package (none) -> Micro-MaTch SMD; Supplier (none) -> Farnell
- P3: Alt. Order Code (none) -> 571-71882756; Alt. Supplier (none) -> Mouser; Note (none) -> 6-way SMD Micro-MaTch connector; Package (none) -> Micro-MaTch SMD; Supplier (none) -> Farnell
- P4: Alt. Order Code (none) -> 571-8-188275-2; Alt. Supplier (none) -> Mouser; Note (none) -> 12-way SMD Micro-MaTch connector; Package (none) -> Micro-MaTch; Supplier (none) -> Farnell
- R1, R2: Alt. Order Code (none) -> 71-CRCW0805-1.5K-E3; Alt. Supplier (none) -> Mouser; Note (none) -> 1.5kΩ/1% 0805 resistor; Package (none) -> 0805; Supplier (none) -> Farnell
- R3, R4, R5: Alt. Order Code (none) -> 71-CRCW0805-100K-E3; Alt. Supplier (none) -> Mouser; Note (none) -> 100kΩ/1% 0805 resistor; Package (none) -> 0805; Supplier (none) -> Farnell
- SHIELD1: Alt. Order Code (none) -> 782-A000062; Alt. Supplier (none) -> Mouser; Manufacturer (none) -> Arduino; Note (none) -> Arduino/Genuino DUE development board; Order Code (none) -> 2250861; Package (none) -> Arduino DUE; Part Number (none) -> A000062; Supplier (none) -> Farnell
- SW1: Alt. Order Code (none) -> 506-FSMRA3JH; Alt. Supplier (none) -> Mouser; Note (none) -> R/A tactile switch; Package (none) -> RA pushbutton; Supplier (none) -> Farnell
- U1: Alt. Order Code (none) -> 579-23LCV1024-I/SN; Alt. Supplier (none) -> Mouser; Note (none) -> 1 Mbit SPI serial SRAM with battery backup and SDI interface; Package (none) -> SOIC-8; Supplier (none) -> Farnell

Commit message: Added MCU power control (MCUswitch.sch)
Parts:
- removed PP12, PP13: CONN_01X01, jakub:PIN_ARRAY_1, symbol CONN_01X01
- added PP29: CONN_01X01, jakub:PIN_ARRAY_1, symbol CONN_01X01
- PP13: renamed from PP15; Supplier (none) -> Farnell
- renumbered PP14 to PP12, PP16 to PP14, PP17 to PP15, PP18 to PP16, PP19 to PP17, PP20 to PP18, PP21 to PP19, PP22 to PP20, PP23 to PP21, PP24 to PP22, PP25 to PP23, PP26 to PP24, PP27 to PP25, PP28 to PP26, PP29 to PP27, PP30 to PP28
Connections:
- net labels added: AD7, PWR_OFF, ~SW_SENSE
- net labels removed: D42, D43, SCLK
- wire segments 181 -> 184
Other:
- moved on the sheet: PP1, PP10, PP11, PP12, PP13, PP14, PP15, PP16, PP17, PP18, PP19, PP2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

Commit message: Finished adding full part descriptions
Parts:
- P5: Alt. Order Code (none) -> SSW-104-02-G-S-RA; Alt. Supplier (none) -> Samtec; Note (none) -> 1x4 right-angle socket strip; Package (none) -> SIL-4; Supplier (none) -> Farnell
- PP13: Supplier Farnell -> (none)
Changed lines of the file:
@@
 F 4 "SSW-104-02-G-S-RA" H 8300 3050 60  0001 C CNN "Part Number"
 F 5 "Samtec" H 8300 3050 60  0001 C CNN "Manufacturer"
-F 6 "1668345" H 8300 3050 60  0001 C CNN "Order Code"
+F 6 "SIL-4" H 8300 3050 60  0001 C CNN "Package"
+F 7 "Farnell" H 8300 3050 60  0001 C CNN "Supplier"
+F 8 "1668345" H 8300 3050 60  0001 C CNN "Order Code"
+F 9 "Samtec" H 8300 3050 60  0001 C CNN "Alt. Supplier"
+F 10 "SSW-104-02-G-S-RA" H 8300 3050 60  0001 C CNN "Alt. Order Code"
+F 11 "1x4 right-angle socket strip" H 8300 3050 60  0001 C CNN "Note"
 	1    8300 3050
 	1    0    0    -1
@@
 F 2 "jakub:PIN_ARRAY_1" H 7300 1100 50  0001 C CNN
 F 3 "" H 7300 1100 50  0000 C CNN
-F 4 "Farnell" H 7300 1100 60  0001 C CNN "Supplier"
 	1    7300 1100
 	1    0    0    -1

Commit message: Incorporated un-pulled changes
Parts:
- A1: renamed from SHIELD1; value ARDUINO_DUE_SHIELD -> Arduino DUE
- P4: Package Micro-MaTch -> Micro-MaTch SMD
- P5: value 1x4 Socket Strip R/A -> 1x4 socket strip R/A
- SW1: value Tactile Switch R/A -> Tactile switch R/A; Note R/A tactile switch -> Right-angle tactile switch; Package RA pushbutton -> R/A pushbutton
Changed lines of the file:
@@
 F 4 "8-188275-2" H 2050 4750 60  0001 C CNN "Part Number"
 F 5 "TE Connectivity" H 2050 4750 60  0001 C CNN "Manufacturer"
-F 6 "Micro-MaTch" H 2050 4750 60  0001 C CNN "Package"
+F 6 "Micro-MaTch SMD" H 2050 4750 60  0001 C CNN "Package"
 F 7 "Farnell" H 2050 4750 60  0001 C CNN "Supplier"
 F 8 "3784757" H 2050 4750 60  0001 C CNN "Order Code"
@@
 P 3700 1700
 F 0 "SW1" H 3850 1810 50  0000 C CNN
-F 1 "Tactile Switch R/A" H 3700 1620 50  0000 C CNN
+F 1 "Tactile switch R/A" H 3700 1620 50  0000 C CNN
 F 2 "jakub:tactileSwitchRA" H 3700 1700 50  0001 C CNN
 F 3 "" H 3700 1700 50  0000 C CNN
 F 4 "MCDTSA6-5N" H 3700 1700 60  0001 C CNN "Part Number"
 F 5 "Multicomp" H 3700 1700 60  0001 C CNN "Manufacturer"
-F 6 "RA pushbutton" H 3700 1700 60  0001 C CNN "Package"
+F 6 "R/A pushbutton" H 3700 1700 60  0001 C CNN "Package"
 F 7 "Farnell" H 3700 1700 60  0001 C CNN "Supplier"
 F 8 "9471804" H 3700 1700 60  0001 C CNN "Order Code"
 F 9 "Mouser" H 3700 1700 60  0001 C CNN "Alt. Supplier"
 F 10 "506-FSMRA3JH" H 3700 1700 60  0001 C CNN "Alt. Order Code"
-F 11 "R/A tactile switch" H 3700 1700 60  0001 C CNN "Note"
+F 11 "Right-angle tactile switch" H 3700 1700 60  0001 C CNN "Note"
 	1    3700 1700
 	0    -1   -1   0
@@
 P 8300 3050
 F 0 "P5" H 8300 3300 50  0000 C CNN
-F 1 "1x4 Socket Strip R/A" V 8400 3050 50  0000 C CNN
+F 1 "1x4 socket strip R/A" V 8400 3050 50  0000 C CNN
 F 2 "Socket_Strips:Socket_Strip_Straight_1x04" H 8300 3050 50  0001 C CNN
 F 3 "" H 8300 3050 50  0000 C CNN
@@
 D32
 $Comp
-L ARDUINO_DUE_SHIELD SHIELD1
+L ARDUINO_DUE_SHIELD A1
 U 1 1 56685571
 P 5700 2950
-F 0 "SHIELD1" H 5100 5300 60  0000 C CNN
-F 1 "ARDUINO_DUE_SHIELD" H 5400 5200 60  0000 C CNN
+F 0 "A1" H 5100 5300 60  0000 L CNN
+F 1 "Arduino DUE" H 5100 5200 60  0000 L CNN
 F 2 "jakub:ARDUINO_DUE" H 5600 2450 60  0001 C CNN
 F 3 "" H 5600 2450 60  0000 C CNN
