File: MicroFLiC_junction_shield.sch (KiCad schematic (older format))
At the start: 45 parts, among them P1 14-way Micro-MaTch, P2 8-way Micro-MaTch, P3 6-way Micro-MaTch, P4 12-way Micro-MaTch, P5 1x4 socket strip R/A, SW1 Tactile switch R/A, U1 23LCV1024

Commit message: Changed LCD shield from Wire to Wire1
Parts:
- added PP20, PP21: CONN_01X01, jakub:PIN_ARRAY_1, symbol CONN_01X01
- renumbered PP20 to PP30, PP21 to PP31
Connections:
- wire segments 184 -> 187
Other:
- moved on the sheet: P3, PP22, PP23, PP24, PP25, PP26, PP27, PP28, PP29, PP30, PP31
