File: humanInterface.sch (KiCad schematic (older format))
At the start: 7 parts, among them Q1 TSM2314, Q2 TSM2314

Commit message: Last commit in v1.0
Parts:
- D1: Manufacturer (none) -> Avago; Order Code (none) -> 8554773; Part Number (none) -> HSMY-C150
Changed lines of the file:
@@
 F 2 "LEDs:LED-1206" H 4700 1600 50  0001 C CNN
 F 3 "" H 4700 1600 50  0000 C CNN
+F 4 "HSMY-C150" H 4700 1600 60  0001 C CNN "Part Number"
+F 5 "Avago" H 4700 1600 60  0001 C CNN "Manufacturer"
+F 6 "8554773" H 4700 1600 60  0001 C CNN "Order Code"
 	1    4700 1600
 	0    -1   -1   0

Commit message: Added MCU power control (MCUswitch.sch)
Parts:
- Q2: Supplier (none) -> Farnell
Changed lines of the file:
@@
 $Descr A4 11693 8268
 encoding utf-8
-Sheet 2 4
+Sheet 2 5
 Title ""
 Date ""
@@
 F 4 "TSM2314CX" H 4600 4900 60  0001 C CNN "Part Number"
 F 5 "Taiwan Semiconductor" H 4600 4900 60  0001 C CNN "Manufacturer"
-F 6 "1864589" H 4600 4900 60  0001 C CNN "Order Code"
+F 6 "Farnell" H 4600 4900 60  0001 C CNN "Supplier"
+F 7 "1864589" H 4600 4900 60  0001 C CNN "Order Code"
 	1    4600 4900
 	1    0    0    -1

Commit message: Finished adding full part descriptions
Parts:
- C4: Alt. Order Code (none) -> 710-885012207098; Alt. Supplier (none) -> Mouser; Note (none) -> 100nF/50V X7R 0805 ceramic capacitor; Package (none) -> 0805; Supplier (none) -> Farnell
- D1: Alt. Order Code (none) -> 630-HSMY-C150; Alt. Supplier (none) -> Mouser; Note (none) -> Yellow 1206 LED; Package (none) -> 1206; Supplier (none) -> Farnell
- Q1: Alt. Order Code (none) -> 781-SI2314EDS-E3; Alt. Supplier (none) -> Mouser; Note (none) -> N-channel SOT-23 MOSFET; Package (none) -> SOT-23; Supplier (none) -> Farnell
- Q2: Alt. Order Code (none) -> 781-SI2314EDS-E3; Alt. Supplier (none) -> Mouser; Note (none) -> N-channel SOT-23 MOSFET; Package (none) -> SOT-23
- R6, R7: Alt. Order Code (none) -> 71-CRCW0805-1.5K-E3; Alt. Supplier (none) -> Mouser; Note (none) -> 1.5kΩ/1% 0805 resistor; Package (none) -> 0805; Supplier (none) -> Farnell
- SP1: Alt. Order Code (none) -> 81-PKM13EPYH4000-A0; Alt. Supplier (none) -> Mouser; Note (none) -> 4kHz piezo sounder; Package (none) -> ⌀12.6mm; Supplier (none) -> Farnell
Changed lines of the file:
@@
 F 4 "HSMY-C150" H 4700 1600 60  0001 C CNN "Part Number"
 F 5 "Avago" H 4700 1600 60  0001 C CNN "Manufacturer"
-F 6 "8554773" H 4700 1600 60  0001 C CNN "Order Code"
+F 6 "1206" H 4700 1600 60  0001 C CNN "Package"
+F 7 "Farnell" H 4700 1600 60  0001 C CNN "Supplier"
+F 8 "8554773" H 4700 1600 60  0001 C CNN "Order Code"
+F 9 "Mouser" H 4700 1600 60  0001 C CNN "Alt. Supplier"
+F 10 "630-HSMY-C150" H 4700 1600 60  0001 C CNN "Alt. Order Code"
+F 11 "Yellow 1206 LED" H 4700 1600 60  0001 C CNN "Note"
 	1    4700 1600
 	0    -1   -1   0
@@
 F 4 "PKM13EPYH4000-A0" H 5300 4100 60  0001 C CNN "Part Number"
 F 5 "Murata" H 5300 4100 60  0001 C CNN "Manufacturer"
-F 6 "1192513" H 5300 4100 60  0001 C CNN "Order Code"
+F 6 "⌀12.6mm" H 5300 4100 60  0001 C CNN "Package"
+F 7 "Farnell" H 5300 4100 60  0001 C CNN "Supplier"
+F 8 "1192513" H 5300 4100 60  0001 C CNN "Order Code"
+F 9 "Mouser" H 5300 4100 60  0001 C CNN "Alt. Supplier"
+F 10 "81-PKM13EPYH4000-A0" H 5300 4100 60  0001 C CNN "Alt. Order Code"
+F 11 "4kHz piezo sounder" H 5300 4100 60  0001 C CNN "Note"
 	1    5300 4100
 	1    0    0    -1
@@
 F 4 "MC0805B104K250CT" H 4400 4250 60  0001 C CNN "Part Number"
 F 5 "Multicomp" H 4400 4250 60  0001 C CNN "Manufacturer"
-F 6 "1759166" H 4400 4250 60  0001 C CNN "Order Code"
+F 6 "0805" H 4400 4250 60  0001 C CNN "Package"
+F 7 "Farnell" H 4400 4250 60  0001 C CNN "Supplier"
+F 8 "1759166" H 4400 4250 60  0001 C CNN "Order Code"
+F 9 "Mouser" H 4400 4250 60  0001 C CNN "Alt. Supplier"
+F 10 "710-885012207098" H 4400 4250 60  0001 C CNN "Alt. Order Code"
+F 11 "100nF/50V X7R 0805 ceramic capacitor" H 4400 4250 60  0001 C CNN "Note"
 	1    4400 4250
 	1    0    0    -1
@@
 F 4 "TSM2314CX" H 4600 2500 60  0001 C CNN "Part Number"
 F 5 "Taiwan Semiconductor" H 4600 2500 60  0001 C CNN "Manufacturer"
-F 6 "1864589" H 4600 2500 60  0001 C CNN "Order Code"
+F 6 "SOT-23" H 4600 2500 60  0001 C CNN "Package"
+F 7 "Farnell" H 4600 2500 60  0001 C CNN "Supplier"
+F 8 "1864589" H 4600 2500 60  0001 C CNN "Order Code"
+F 9 "Mouser" H 4600 2500 60  0001 C CNN "Alt. Supplier"
+F 10 "781-SI2314EDS-E3" H 4600 2500 60  0001 C CNN "Alt. Order Code"
+F 11 "N-channel SOT-23 MOSFET" H 4600 2500 60  0001 C CNN "Note"
 	1    4600 2500
 	1    0    0    -1
@@
 F 4 "TSM2314CX" H 4600 4900 60  0001 C CNN "Part Number"
 F 5 "Taiwan Semiconductor" H 4600 4900 60  0001 C CNN "Manufacturer"
-F 6 "Farnell" H 4600 4900 60  0001 C CNN "Supplier"
-F 7 "1864589" H 4600 4900 60  0001 C CNN "Order Code"
+F 6 "SOT-23" H 4600 4900 60  0001 C CNN "Package"
+F 7 "Farnell" H 4600 4900 60  0001 C CNN "Supplier"
+F 8 "1864589" H 4600 4900 60  0001 C CNN "Order Code"
+F 9 "Mouser" H 4600 4900 60  0001 C CNN "Alt. Supplier"
+F 10 "781-SI2314EDS-E3" H 4600 4900 60  0001 C CNN "Alt. Order Code"
+F 11 "N-channel SOT-23 MOSFET" H 4600 4900 60  0001 C CNN "Note"
 	1    4600 4900
 	1    0    0    -1
@@
 F 4 "MCWR08X1501FTL" V 4700 2050 60  0001 C CNN "Part Number"
 F 5 "Multicomp" V 4700 2050 60  0001 C CNN "Manufacturer"
-F 6 "2447592" V 4700 2050 60  0001 C CNN "Order Code"
+F 6 "0805" H 4700 2050 60  0001 C CNN "Package"
+F 7 "Farnell" H 4700 2050 60  0001 C CNN "Supplier"
+F 8 "2447592" V 4700 2050 60  0001 C CNN "Order Code"
+F 9 "Mouser" H 4700 2050 60  0001 C CNN "Alt. Supplier"
+F 10 "71-CRCW0805-1.5K-E3" H 4700 2050 60  0001 C CNN "Alt. Order Code"
+F 11 "1.5kΩ/1% 0805 resistor" H 4700 2050 60  0001 C CNN "Note"
 	1    4700 2050
 	1    0    0    -1
@@
 F 4 "MCWR08X1501FTL" V 4700 4250 60  0001 C CNN "Part Number"
 F 5 "Multicomp" V 4700 4250 60  0001 C CNN "Manufacturer"
-F 6 "2447592" V 4700 4250 60  0001 C CNN "Order Code"
+F 6 "0805" H 4700 4250 60  0001 C CNN "Package"
+F 7 "Farnell" H 4700 4250 60  0001 C CNN "Supplier"
+F 8 "2447592" V 4700 4250 60  0001 C CNN "Order Code"
+F 9 "Mouser" H 4700 4250 60  0001 C CNN "Alt. Supplier"
+F 10 "71-CRCW0805-1.5K-E3" H 4700 4250 60  0001 C CNN "Alt. Order Code"
+F 11 "1.5kΩ/1% 0805 resistor" H 4700 4250 60  0001 C CNN "Note"
 	1    4700 4250
 	1    0    0    -1

Commit message: Changed part number or yellow LED
Parts:
- D1: Order Code 8554773 -> 2497382
Changed lines of the file:
@@
 F 6 "1206" H 4700 1600 60  0001 C CNN "Package"
 F 7 "Farnell" H 4700 1600 60  0001 C CNN "Supplier"
-F 8 "8554773" H 4700 1600 60  0001 C CNN "Order Code"
+F 8 "2497382" H 4700 1600 60  0001 C CNN "Order Code"
 F 9 "Mouser" H 4700 1600 60  0001 C CNN "Alt. Supplier"
 F 10 "630-HSMY-C150" H 4700 1600 60  0001 C CNN "Alt. Order Code"

Commit message: Incorporated un-pulled changes
Parts:
- SP1: value PIEZO SOUNDER -> Piezo sounder
Changed lines of the file:
@@
 P 5300 4100
 F 0 "SP1" H 5200 4350 50  0000 C CNN
-F 1 "PIEZO SOUNDER" H 5300 3750 50  0000 C CNN
+F 1 "Piezo sounder" H 5300 3750 50  0000 C CNN
 F 2 "jakub:piezo" H 5300 4100 50  0001 C CNN
 F 3 "" H 5300 4100 50  0000 C CNN

Commit message: Changed SHIELD1 to A1, changed SOD-323 footprint for easier soldering
Parts:
- D1: Manufacturer Avago -> Broadcom
Changed lines of the file:
@@
 F 3 "" H 4700 1600 50  0000 C CNN
 F 4 "HSMY-C150" H 4700 1600 60  0001 C CNN "Part Number"
-F 5 "Avago" H 4700 1600 60  0001 C CNN "Manufacturer"
+F 5 "Broadcom" H 4700 1600 60  0001 C CNN "Manufacturer"
 F 6 "1206" H 4700 1600 60  0001 C CNN "Package"
 F 7 "Farnell" H 4700 1600 60  0001 C CNN "Supplier"
