File: pins.sch (KiCad schematic (older format))
At the start: 20 parts, among them P10 1x8 header strip, P11 1x8 header strip, P12 1x8 header strip, P13 1x10 header strip, P14 2x3 socket strip, P7 2x18 header strip, P8 1x8 header strip, P9 1x8 header strip

Commit message: Changed LCD shield from Wire to Wire1
Parts:
- renumbered PP30 to PP42, PP31 to PP43
Connections:
- net +3V3: now also PP33.1 (P1), PP34.1 (P1); no longer PP42.1 (P1), PP43.1 (P1)
- net +5V: now also PP36.1 (P1), PP37.1 (P1); no longer PP33.1 (P1), PP34.1 (P1)
- net GND: now also PP42.1 (P1), PP43.1 (P1); no longer PP36.1 (P1), PP37.1 (P1)
Other:
- moved on the sheet: PP32, PP33, PP34, PP35, PP36, PP37, PP38, PP39, PP40, PP41, PP42, PP43
Changed lines of the file:
@@
 EESchema Schematic File Version 2
-LIBS:MicroFLiC_junction_shield-rescue
 LIBS:power
 LIBS:device
@@
 $EndDescr
 $Comp
-L CONN_01X01 PP31
+L CONN_01X01 PP43
 U 1 1 566CC01D
+P 4450 3200
+F 0 "PP43" H 4550 3200 50  0000 L CNN
+F 1 "CONN_01X01" V 4550 3200 50  0001 C CNN
+F 2 "jakub:PIN_ARRAY_1" H 4450 3200 50  0001 C CNN
+F 3 "" H 4450 3200 50  0000 C CNN
+	1    4450 3200
+	1    0    0    -1
+$EndComp
+$Comp
+L CONN_01X01 PP32
+U 1 1 566CC024
+P 4450 1600
+F 0 "PP32" H 4550 1600 50  0000 L CNN
+F 1 "CONN_01X01" V 4550 1600 50  0001 C CNN
+F 2 "jakub:PIN_ARRAY_1" H 4450 1600 50  0001 C CNN
+F 3 "" H 4450 1600 50  0000 C CNN
+	1    4450 1600
+	1    0    0    -1
+$EndComp
+$Comp
+L CONN_01X01 PP33
+U 1 1 566CC02B
 P 4450 1700
-F 0 "PP31" H 4550 1700 50  0000 L CNN
+F 0 "PP33" H 4550 1700 50  0000 L CNN
 F 1 "CONN_01X01" V 4550 1700 50  0001 C CNN
 F 2 "jakub:PIN_ARRAY_1" H 4450 1700 50  0001 C CNN
@@
 	1    0    0    -1
 $EndComp
-$Comp
-L CONN_01X01 PP32
-U 1 1 566CC024
+Wire Wire Line
+	4150 1800 4250 1800
+Wire Wire Line
+	4150 1500 4150 1800
+Wire Wire Line
+	4150 1700 4250 1700
+Wire Wire Line
+	4150 1600 4250 1600
+Connection ~ 4150 1700
+Connection ~ 4150 1600
+Wire Wire Line
+	4150 2400 4250 2400
+Wire Wire Line
+	4150 2100 4150 2400
+Wire Wire Line
+	4150 2300 4250 2300
+Wire Wire Line
+	4150 2200 4250 2200
+Connection ~ 4150 2300
+Connection ~ 4150 2200
+Wire Wire Line
+	4250 2700 4150 2700
+Wire Wire Line
+	4150 2700 4150 3300
+Wire Wire Line
+	4150 2800 4250 2800
+Wire Wire Line
+	4150 2900 4250 2900
+Connection ~ 4150 2800
+Connection ~ 4150 2900
+$Comp
+L GND #PWR044
+U 1 1 566CC06E
+P 4150 3300
+F 0 "#PWR044" H 4150 3050 50  0001 C CNN
+F 1 "GND" H 4150 3150 50  0000 C CNN
+F 2 "" H 4150 3300 50  0000 C CNN
+F 3 "" H 4150 3300 50  0000 C CNN
+	1    4150 3300
+	1    0    0    -1
+$EndComp
+$Comp
+L +5V #PWR045
+U 1 1 566CC074
+P 4150 2100
+F 0 "#PWR045" H 4150 1950 50  0001 C CNN
+F 1 "+5V" H 4150 2240 50  0000 C CNN
+F 2 "" H 4150 2100 50  0000 C CNN
+F 3 "" H 4150 2100 50  0000 C CNN
+	1    4150 2100
+	1    0    0    -1
+$EndComp
+$Comp
+L +3V3 #PWR046
+U 1 1 566CC07A
+P 4150 1500
+F 0 "#PWR046" H 4150 1350 50  0001 C CNN
+F 1 "+3V3" H 4150 1640 50  0000 C CNN
+F 2 "" H 4150 1500 50  0000 C CNN
+F 3 "" H 4150 1500 50  0000 C CNN
+	1    4150 1500
+	1    0    0    -1
+$EndComp
+Wire Wire Line
+	4150 3000 4250 3000
+Wire Wire Line
+	4150 3100 4250 3100
+Wire Wire Line
+	4150 3200 4250 3200
+Connection ~ 4150 3100
+Connection ~ 4150 3200
+Connection ~ 4150 3000
+$Comp
+L CONN_01X01 PP34
+U 1 1 5671D822
 P 4450 1800
-F 0 "PP32" H 4550 1800 50  0000 L CNN
+F 0 "PP34" H 4550 1800 50  0000 L CNN
 F 1 "CONN_01X01" V 4550 1800 50  0001 C CNN
 F 2 "jakub:PIN_ARRAY_1" H 4450 1800 50  0001 C CNN
@@
 $EndComp
 $Comp
-L CONN_01X01 PP33
-U 1 1 566CC02B
+L CONN_01X01 PP35
+U 1 1 5671D828
 P 4450 2200
-F 0 "PP33" H 4550 2200 50  0000 L CNN
+F 0 "PP35" H 4550 2200 50  0000 L CNN
 F 1 "CONN_01X01" V 4550 2200 50  0001 C CNN
 F 2 "jakub:PIN_ARRAY_1" H 4450 2200 50  0001 C CNN
@@
 	1    0    0    -1
 $EndComp
-Wire Wire Line
-	4150 1800 4250 1800
-Wire Wire Line
-	4150 1500 4150 1800
-Wire Wire Line
-	4150 1700 4250 1700
-Wire Wire Line
-	4150 1600 4250 1600
-Connection ~ 4150 1700
-Connection ~ 4150 1600
-Wire Wire Line
-	4150 2400 4250 2400
-Wire Wire Line
-	4150 2100 4150 2400
-Wire Wire Line
-	4150 2300 4250 2300
-Wire Wire Line
-	4150 2200 4250 2200
-Connection ~ 4150 2300
-Connection ~ 4150 2200
-Wire Wire Line
-	4250 2700 4150 2700
-Wire Wire Line
-	4150 2700 4150 3300
-Wire Wire Line
-	4150 2800 4250 2800
-Wire Wire Line
-	4150 2900 4250 2900
-Connection ~ 4150 2800
-Connection ~ 4150 2900
-$Comp
-L GND #PWR42
-U 1 1 566CC06E
-P 4150 3300
-F 0 "#PWR42" H 4150 3050 50  0001 C CNN
-F 1 "GND" H 4150 3150 50  0000 C CNN
-F 2 "" H 4150 3300 50  0000 C CNN
-F 3 "" H 4150 3300 50  0000 C CNN
-	1    4150 3300
-	1    0    0    -1
-$EndComp
-$Comp
-L +5V #PWR41
-U 1 1 566CC074
-P 4150 2100
-F 0 "#PWR41" H 4150 1950 50  0001 C CNN
-F 1 "+5V" H 4150 2240 50  0000 C CNN
-F 2 "" H 4150 2100 50  0000 C CNN
-F 3 "" H 4150 2100 50  0000 C CNN
-	1    4150 2100
-	1    0    0    -1
-$EndComp
-$Comp
-L +3V3 #PWR40
-U 1 1 566CC07A
-P 4150 1500
-F 0 "#PWR40" H 4150 1350 50  0001 C CNN
-F 1 "+3V3" H 4150 1640 50  0000 C CNN
-F 2 "" H 4150 1500 50  0000 C CNN
-F 3 "" H 4150 1500 50  0000 C CNN
-	1    4150 1500
-	1    0    0    -1
-$EndComp
-Wire Wire Line
-	4150 3000 4250 3000
-Wire Wire Line
-	4150 3100 4250 3100
-Wire Wire Line
-	4150 3200 4250 3200
-Connection ~ 4150 3100
-Connection ~ 4150 3200
-Connection ~ 4150 3000
-$Comp
-L CONN_01X01 PP34
-U 1 1 5671D822
+$Comp
+L CONN_01X01 PP36
+U 1 1 5671D82E
 P 4450 2300
-F 0 "PP34" H 4550 2300 50  0000 L CNN
+F 0 "PP36" H 4550 2300 50  0000 L CNN
 F 1 "CONN_01X01" V 4550 2300 50  0001 C CNN
 F 2 "jakub:PIN_ARRAY_1" H 4450 2300 50  0001 C CNN
@@
 $EndComp
 $Comp
-L CONN_01X01 PP35
-U 1 1 5671D828
+L CONN_01X01 PP37
+U 1 1 5671D8A0
 P 4450 2400
-F 0 "PP35" H 4550 2400 50  0000 L CNN
+F 0 "PP37" H 4550 2400 50  0000 L CNN
 F 1 "CONN_01X01" V 4550 2400 50  0001 C CNN
 F 2 "jakub:PIN_ARRAY_1" H 4450 2400 50  0001 C CNN
@@
 $EndComp
 $Comp
-L CONN_01X01 PP36
-U 1 1 5671D82E
+L CONN_01X01 PP38
+U 1 1 5671D8A6
 P 4450 2700
-F 0 "PP36" H 4550 2700 50  0000 L CNN
+F 0 "PP38" H 4550 2700 50  0000 L CNN
 F 1 "CONN_01X01" V 4550 2700 50  0001 C CNN
 F 2 "jakub:PIN_ARRAY_1" H 4450 2700 50  0001 C CNN
@@
 $EndComp
 $Comp
-L CONN_01X01 PP37
-U 1 1 5671D8A0
+L CONN_01X01 PP39
+U 1 1 5671D8AC
 P 4450 2800
-F 0 "PP37" H 4550 2800 50  0000 L CNN
+F 0 "PP39" H 4550 2800 50  0000 L CNN
 F 1 "CONN_01X01" V 4550 2800 50  0001 C CNN
 F 2 "jakub:PIN_ARRAY_1" H 4450 2800 50  0001 C CNN
@@
 $EndComp
 $Comp
-L CONN_01X01 PP38
-U 1 1 5671D8A6
+L CONN_01X01 PP40
+U 1 1 5671D918
 P 4450 2900
-F 0 "PP38" H 4550 2900 50  0000 L CNN
+F 0 "PP40" H 4550 2900 50  0000 L CNN
 F 1 "CONN_01X01" V 4550 2900 50  0001 C CNN
 F 2 "jakub:PIN_ARRAY_1" H 4450 2900 50  0001 C CNN
@@
 $EndComp
 $Comp
-L CONN_01X01 PP39
-U 1 1 5671D8AC
+L CONN_01X01 PP41
+U 1 1 5671D91E
 P 4450 3000
-F 0 "PP39" H 4550 3000 50  0000 L CNN
+F 0 "PP41" H 4550 3000 50  0000 L CNN
 F 1 "CONN_01X01" V 4550 3000 50  0001 C CNN
 F 2 "jakub:PIN_ARRAY_1" H 4450 3000 50  0001 C CNN
@@
 $EndComp
 $Comp
-L CONN_01X01 PP40
-U 1 1 5671D918
+L CONN_01X01 PP42
+U 1 1 5671D924
 P 4450 3100
-F 0 "PP40" H 4550 3100 50  0000 L CNN
+F 0 "PP42" H 4550 3100 50  0000 L CNN
 F 1 "CONN_01X01" V 4550 3100 50  0001 C CNN
 F 2 "jakub:PIN_ARRAY_1" H 4450 3100 50  0001 C CNN
@@
 	1    0    0    -1
 $EndComp
-$Comp
-L CONN_01X01 PP41
-U 1 1 5671D91E
-P 4450 3200
-F 0 "PP41" H 4550 3200 50  0000 L CNN
-F 1 "CONN_01X01" V 4550 3200 50  0001 C CNN
-F 2 "jakub:PIN_ARRAY_1" H 4450 3200 50  0001 C CNN
-F 3 "" H 4450 3200 50  0000 C CNN
-	1    4450 3200
-	1    0    0    -1
-$EndComp
-$Comp
-L CONN_01X01 PP30
-U 1 1 5671D924
-P 4450 1600
-F 0 "PP30" H 4550 1600 50  0000 L CNN
-F 1 "CONN_01X01" V 4550 1600 50  0001 C CNN
-F 2 "jakub:PIN_ARRAY_1" H 4450 1600 50  0001 C CNN
-F 3 "" H 4450 1600 50  0000 C CNN
-	1    4450 1600
-	1    0    0    -1
-$EndComp
